File: PCB/splitflap_01.sch (EAGLE design)
At the start: 22 parts, among them IC2 ULN2003AD, U1 ATTINY84

Commit message: 1. Vorschlag by happyprinter
Connections:
- net A: now also U1.(ADC0)PA0; no longer U1.(ADC3)PA3
- net B: now also U1.(ADC1)PA1; no longer U1.(ADC2)PA2
- net C: now also U1.(ADC2)PA2; no longer U1.(ADC1)PA1
- net D: now also U1.(ADC3)PA3; no longer U1.(ADC0)PA0
Changed lines of the file:
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@@
 <setting verticaltext="up"/>
 </settings>
-<grid distance="0.1" unitdist="inch" unit="inch" style="lines" multiple="1" display="yes" altdistance="0.01" altunitdist="inch" altunit="inch"/>
+<grid distance="0.1" unitdist="inch" unit="inch" style="lines" multiple="1" display="no" altdistance="0.01" altunitdist="inch" altunit="inch"/>
 <layers>
 <layer number="1" name="Top" color="4" fill="1" visible="no" active="no"/>
@@
 </segment>
 <segment>
-<pinref part="U1" gate="U1" pin="(ADC3)PA3"/>
-<wire x1="81.28" y1="88.9" x2="83.82" y2="88.9" width="0.4064" layer="91"/>
-<label x="83.82" y="88.9" size="1.778" layer="95"/>
+<pinref part="U1" gate="U1" pin="(ADC0)PA0"/>
+<wire x1="81.28" y1="81.28" x2="83.82" y2="81.28" width="0.1524" layer="91"/>
+<label x="84.582" y="80.518" size="1.778" layer="95"/>
 </segment>
 </net>
@@
 </segment>
 <segment>
-<pinref part="U1" gate="U1" pin="(ADC2)PA2"/>
-<wire x1="81.28" y1="86.36" x2="83.82" y2="86.36" width="0.4064" layer="91"/>
-<label x="83.82" y="86.36" size="1.778" layer="95"/>
+<pinref part="U1" gate="U1" pin="(ADC1)PA1"/>
+<wire x1="81.28" y1="83.82" x2="83.82" y2="83.82" width="0.1524" layer="91"/>
+<label x="84.582" y="82.804" size="1.778" layer="95"/>
 </segment>
 </net>
@@
 </segment>
 <segment>
-<pinref part="U1" gate="U1" pin="(ADC1)PA1"/>
-<wire x1="81.28" y1="83.82" x2="83.82" y2="83.82" width="0.4064" layer="91"/>
-<label x="83.82" y="83.82" size="1.778" layer="95"/>
+<pinref part="U1" gate="U1" pin="(ADC2)PA2"/>
+<wire x1="81.28" y1="86.36" x2="83.82" y2="86.36" width="0.1524" layer="91"/>
+<label x="84.582" y="85.598" size="1.778" layer="95"/>
 </segment>
 </net>
@@
 </segment>
 <segment>
-<pinref part="U1" gate="U1" pin="(ADC0)PA0"/>
-<wire x1="81.28" y1="81.28" x2="83.82" y2="81.28" width="0.4064" layer="91"/>
-<label x="83.82" y="81.28" size="1.778" layer="95"/>
-</segment>
-</net>
+<pinref part="U1" gate="U1" pin="(ADC3)PA3"/>
+<wire x1="81.28" y1="88.9" x2="83.82" y2="88.9" width="0.1524" layer="91"/>
+<label x="84.582" y="88.138" size="1.778" layer="95"/>
+</segment>
+</net>
