File: PCB/splitflap_01.brd (EAGLE design)
At the start: 51 x 26 mm, 22 parts, among them IC2 ULN2003AD, U1 ATTINY84

Commit message: 1. Vorschlag by happyprinter
Parts:
- moved IC3 40.3 mm to (45.5, 19.5), turned to 0 degrees
- moved C1 36.2 mm to (43.5, 13.5), turned to 180 degrees
- moved C5 32.0 mm to (45.5, 9.50), turned to 180 degrees
- moved C3 16.8 mm to (4.00, 5.00), turned to 180 degrees
- moved + 16.0 mm to (33.5, 23.0)
- moved R2 14.0 mm to (27.0, 3.50)
- moved U1 12.1 mm to (33.0, 14.0), turned to 180 degrees
- moved C4 11.5 mm to (26.0, 13.0)
- moved IC2 10.5 mm to (19.5, 13.0)
- moved R1 8.02 mm to (36.0, 3.50)
- moved C2 7.43 mm to (39.5, 14.0), turned to 270 degrees
- moved P1 4.00 mm to (17.5, 23.0)
- moved P2 4.00 mm to (21.5, 23.0)
- moved P3 4.00 mm to (25.5, 23.0)
- moved P4 4.00 mm to (29.5, 23.0)
Connections:
- net A: now also U1.13; no longer U1.10
- net B: now also U1.12; no longer U1.11
- net C: now also U1.11; no longer U1.12
- net D: now also U1.10; no longer U1.13
Routing:
- net +12V: track 0.00 -> 100.3 mm
- net HALL_SENSOR: track 0.00 -> 41.4 mm, vias 0 -> 1
- net GND: track 0.00 -> 27.1 mm, vias 0 -> 39
- net A: track 0.00 -> 25.7 mm
- net B: track 0.00 -> 22.0 mm
- net N$1: track 0.00 -> 22.0 mm, vias 0 -> 2
- net +3V3: track 0.00 -> 19.5 mm
- net C: track 0.00 -> 18.7 mm
- net N$2: track 0.00 -> 15.5 mm, vias 0 -> 2
- net D: track 0.00 -> 15.3 mm
- net N$6: track 0.00 -> 15.1 mm
- net N$5: track 0.00 -> 13.7 mm
- net N$4: track 0.00 -> 10.2 mm
- net N$3: track 0.00 -> 7.94 mm
- net SCL: track 0.00 -> 3.02 mm
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- added copper zone on layer 1, net GND

Commit message: 2. Version by Happyprinter
Parts:
- moved C2 0.50 mm to (39.5, 13.5)
- moved C4 0.50 mm to (26.0, 13.5)
- moved IC2 0.50 mm to (19.5, 13.5)
- moved R1 0.50 mm to (36.5, 3.50)
- moved R2 0.50 mm to (26.5, 3.50)
- moved U1 0.50 mm to (33.0, 13.5)
Routing:
- net GND: track 27.1 -> 19.9 mm, vias 39 -> 64
- net N$1: track 22.0 -> 23.3 mm
- net +12V: track 100.3 -> 99.8 mm
- net SDA: track 3.02 -> 3.52 mm
- net SCL: track 3.02 -> 3.52 mm
- net N$5: track 13.7 -> 13.2 mm
- net N$3: track 7.94 -> 7.44 mm
- net HALL_SENSOR: track 41.4 -> 40.9 mm
