File: PCB/splitflap_02.brd (EAGLE design)
At the start: 51 x 26 mm, 14 parts, among them IC2 ULN2003AD, U1 ATTINY84, X2 S5B-XH-A

Commit message: Schön layoutete Version by Happyprinter
Parts:
- moved R2 7.16 mm to (34.5, 9.00), turned to 270 degrees
- moved R1 5.15 mm to (32.8, 9.00), turned to 270 degrees
- moved U1 5.13 mm to (22.2, 16.5)
- moved JP1 4.87 mm to (28.6, 15.9), turned to 90 degrees
- moved C1 4.16 mm to (23.8, 10.5)
- moved C4 1.68 mm to (11.2, 22.5)
- moved IC2 1.68 mm to (11.2, 15.5)
- moved C5 0.25 mm to (16.2, 5.00)
Routing:
- net GND: track 81.5 -> 0.32 mm, vias 0 -> 62
- net SCK: track 76.4 -> 44.2 mm
- net MOSI: track 50.6 -> 21.4 mm
- net +3V3: track 41.2 -> 15.6 mm
- net HALL_SENSOR: track 58.0 -> 48.2 mm
- net RESET: track 12.8 -> 5.37 mm
- net D: track 13.0 -> 7.50 mm
- net B: track 13.0 -> 7.50 mm
- net A: track 13.0 -> 7.50 mm
- net C: track 13.0 -> 7.50 mm
- net SCL: track 6.51 -> 11.5 mm
- net N$5: track 10.4 -> 6.77 mm
- net N$4: track 11.7 -> 8.23 mm
- net N$6: track 9.19 -> 6.26 mm
- net N$3: track 12.9 -> 9.98 mm
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